File: hw/open-lion-charger/Charge.kicad_sch (KiCad schematic)
At the start: 40 parts, among them IC6 LM5170QPHPTQ1

Commit message: Done with PCB review
Warning : issue with net +12P and confusion with RELAIS_BATT_OUT
Parts:
- IC6: footprint libTX54:QFP50P900X900X120-49N -> open-lion:QFP50P900X900X120-49N
Changed lines of the file:
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@@
 			)
 		)
-		(property "Footprint" "libTX54:QFP50P900X900X120-49N"
+		(property "Footprint" "open-lion:QFP50P900X900X120-49N"
 			(at 167.894 66.548 0)
 			(effects
