File: hw/open-lion-charger/Charge_Phases.kicad_sch (KiCad schematic)
At the start: 34 parts, among them Q10 PSMNR55-40SSHJ, Q11 PSMNR55-40SSHJ, Q12 PSMNR55-40SSHJ, Q13 PSMNR55-40SSHJ, Q14 PSMNR55-40SSHJ, Q5 PSMNR55-40SSHJ, Q6 PSMNR55-40SSHJ, Q9 PSMNR55-40SSHJ

Commit message: Done with PCB review
Warning : issue with net +12P and confusion with RELAIS_BATT_OUT
Parts:
- L1, L2: footprint libTX54:B82559A6472A024 -> open-lion:B82559A6472A024
- Q10, Q11, Q12, Q13, Q14, Q5, Q6, Q9: footprint libTX54:LFPAK88 -> open-lion:LFPAK88
- R34, R43: footprint GKM5R0010FETR -> open-lion:WSLP40261L000FEA
Changed lines of the file:
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@@
 			)
 		)
-		(property "Footprint" "libTX54:LFPAK88"
+		(property "Footprint" "open-lion:LFPAK88"
 			(at 115.57 46.99 0)
 			(effects
@@
 			)
 		)
-		(property "Footprint" "libTX54:LFPAK88"
+		(property "Footprint" "open-lion:LFPAK88"
 			(at 132.08 31.75 0)
 			(effects
@@
 			)
 		)
-		(property "Footprint" "libTX54:LFPAK88"
+		(property "Footprint" "open-lion:LFPAK88"
 			(at 167.64 49.53 0)
 			(effects
@@
 			)
 		)
-		(property "Footprint" "libTX54:LFPAK88"
+		(property "Footprint" "open-lion:LFPAK88"
 			(at 151.13 63.5 0)
 			(effects
@@
 			)
 		)
-		(property "Footprint" "libTX54:B82559A6472A024"
+		(property "Footprint" "open-lion:B82559A6472A024"
 			(at 189.23 31.75 0)
 			(effects
@@
 			)
 		)
-		(property "Footprint" "GKM5R0010FETR"
+		(property "Footprint" "open-lion:WSLP40261L000FEA"
 			(at 209.55 34.29 0)
 			(effects
@@
 			)
 		)
-		(property "Footprint" "libTX54:LFPAK88"
+		(property "Footprint" "open-lion:LFPAK88"
 			(at 115.57 121.92 0)
 			(effects
@@
 			)
 		)
-		(property "Footprint" "libTX54:LFPAK88"
+		(property "Footprint" "open-lion:LFPAK88"
 			(at 132.08 106.68 0)
 			(effects
@@
 			)
 		)
-		(property "Footprint" "libTX54:LFPAK88"
+		(property "Footprint" "open-lion:LFPAK88"
 			(at 167.64 124.46 0)
 			(effects
@@
 			)
 		)
-		(property "Footprint" "libTX54:LFPAK88"
+		(property "Footprint" "open-lion:LFPAK88"
 			(at 151.13 138.43 0)
 			(effects
@@
 			)
 		)
-		(property "Footprint" "libTX54:B82559A6472A024"
+		(property "Footprint" "open-lion:B82559A6472A024"
 			(at 189.23 106.68 0)
 			(effects
@@
 			)
 		)
-		(property "Footprint" "GKM5R0010FETR"
+		(property "Footprint" "open-lion:WSLP40261L000FEA"
 			(at 222.25 104.14 0)
 			(effects
