File: hw/open-lion-charger/Charge_control.kicad_sch (KiCad schematic)
At the start: 39 parts, among them IC10 MUX509IDR, IC5 INA280A3IDCKR, U4 TLV9151SIDBVR, U5 TLV9151SIDBVR, U8 AD5663BRMZ-1

Commit message: Done with PCB review
Warning : issue with net +12P and confusion with RELAIS_BATT_OUT
Parts:
- IC10: footprint SOIC127P600X175-16N -> open-lion:SOIC127P600X175-16N
- IC5: footprint SOT65P210X110-5N -> open-lion:SOT65P210X110-5N
- R25: footprint GKM5R0010FETR -> open-lion:WSLP40261L000FEA
- U8: footprint libTX54:AD5663BRMZ-1 -> open-lion:AD5663BRMZ-1
Changed lines of the file:
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@@
 			)
 		)
-		(property "Footprint" "SOIC127P600X175-16N"
+		(property "Footprint" "open-lion:SOIC127P600X175-16N"
 			(at 190.5 86.36 0)
 			(effects
@@
 			)
 		)
-		(property "Footprint" "libTX54:AD5663BRMZ-1"
+		(property "Footprint" "open-lion:AD5663BRMZ-1"
 			(at 222.504 17.78 0)
 			(effects
@@
 			)
 		)
-		(property "Footprint" "GKM5R0010FETR"
+		(property "Footprint" "open-lion:WSLP40261L000FEA"
 			(at 65.405 146.939 0)
 			(effects
@@
 			)
 		)
-		(property "Footprint" "SOT65P210X110-5N"
+		(property "Footprint" "open-lion:SOT65P210X110-5N"
 			(at 50.165 169.545 0)
 			(effects
