File: hw/open-lion-charger/Data_Sensors.kicad_sch (KiCad schematic)
At the start: 42 parts, among them IC2 DS3231M+TRL, IC3 TMP36GRTZ-REEL7, IC4 ADS122C04IPWR, J5 Conn_01x02_Female, J6 Conn_01x02_Female, U2 MAX31855JASA, U3 MAX31855JASA, U9 MAX3377EEUD+

Commit message: Done with PCB review
Warning : issue with net +12P and confusion with RELAIS_BATT_OUT
Parts:
- IC2: footprint SOIC127P1032X265-16N -> open-lion:SOIC127P1032X265-16N
- IC3: footprint SOT95P280X145-5N -> open-lion:SOT95P280X145-5N
- IC4: footprint libTX54:SOP65P640X120-16N -> open-lion:SOP65P640X120-16N
Changed lines of the file:
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@@
 			)
 		)
-		(property "Footprint" "SOIC127P1032X265-16N"
+		(property "Footprint" "open-lion:SOIC127P1032X265-16N"
 			(at 92.964 20.32 0)
 			(effects
@@
 			)
 		)
-		(property "Footprint" "SOT95P280X145-5N"
+		(property "Footprint" "open-lion:SOT95P280X145-5N"
 			(at 99.822 98.171 0)
 			(effects
@@
 			)
 		)
-		(property "Footprint" "libTX54:SOP65P640X120-16N"
+		(property "Footprint" "open-lion:SOP65P640X120-16N"
 			(at 208.788 28.702 0)
 			(effects
