File: hw/open-lion-charger/Discharge.kicad_sch (KiCad schematic)
At the start: 21 parts, among them IC7 INA280A3IDCKR, IC8 INA280A3IDCKR, IC9 DAC80501MDGSR, Q7 IXTH30N50L2, Q8 IXTH30N50L2, U6 LMP7701, U7 LMP7701

Commit message: Done with PCB review
Warning : issue with net +12P and confusion with RELAIS_BATT_OUT
Parts:
- IC7, IC8: footprint SOT65P210X110-5N -> open-lion:SOT65P210X110-5N
- IC9: footprint libTX54:SOP50P490X110-10N -> open-lion:SOP50P490X110-10N
- R36, R37: footprint GKM5R0010FETR -> open-lion:WSLP40261L000FEA
Changed lines of the file:
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@@
 			)
 		)
-		(property "Footprint" "libTX54:SOP50P490X110-10N"
+		(property "Footprint" "open-lion:SOP50P490X110-10N"
 			(at 247.142 60.071 0)
 			(effects
@@
 			)
 		)
-		(property "Footprint" "GKM5R0010FETR"
+		(property "Footprint" "open-lion:WSLP40261L000FEA"
 			(at 118.872 112.268 0)
 			(effects
@@
 			)
 		)
-		(property "Footprint" "GKM5R0010FETR"
+		(property "Footprint" "open-lion:WSLP40261L000FEA"
 			(at 170.688 112.395 0)
 			(effects
@@
 			)
 		)
-		(property "Footprint" "SOT65P210X110-5N"
+		(property "Footprint" "open-lion:SOT65P210X110-5N"
 			(at 103.632 134.874 0)
 			(effects
@@
 			)
 		)
-		(property "Footprint" "SOT65P210X110-5N"
+		(property "Footprint" "open-lion:SOT65P210X110-5N"
 			(at 155.448 135.001 0)
 			(effects
