File: hw/open-lion-charger/open-lion-charger.kicad_pcb (KiCad board)
At the start: 2 copper layers, 139.7 x 186 mm, 235 parts, among them IC1 MCP1799-3302H_DB, IC10 MUX509IDR, IC2 DS3231M+TRL, IC3 TMP36GRTZ-REEL7, IC4 ADS122C04IPWR, IC5 INA280A3IDCKR, IC6 LM5170QPHPTQ1, IC7 INA280A3IDCKR, IC8 INA280A3IDCKR, IC9 DAC80501MDGSR, J1 Barrel_Jack_Switch, J2 Conn_01x02_Female, J3 Conn_01x02_Female, J4 Conn_01x06_Female, J5 Conn_01x02_Female, J6 Conn_01x02_Female, J8 Conn_01x02_Female, J9 USB_C_Receptacle, K1 G6QE-1A_DC12, P1 Power, P2 Analog, P3 Digital, P4 Digital, Q1 PBHV9115TLH, Q10 PSMNR55-40SSHJ, Q11 PSMNR55-40SSHJ, Q12 PSMNR55-40SSHJ, Q13 PSMNR55-40SSHJ, Q14 PSMNR55-40SSHJ, Q2 SiS176LDN, Q3 PBHV8115T, Q4 PBHV8115T, Q5 PSMNR55-40SSHJ, Q6 PSMNR55-40SSHJ, Q7 IXTH30N50L2, Q8 IXTH30N50L2, Q9 PSMNR55-40SSHJ, U1 LM1117-5.0, U10 FUSB302T, U2 MAX31855JASA, U3 MAX31855JASA, U4 TLV9151SIDBVR, U5 TLV9151SIDBVR, U6 LMP7701, U7 LMP7701, U8 AD5663BRMZ-1, U9 MAX3377EEUD+

Commit message: Done with PCB review
Warning : issue with net +12P and confusion with RELAIS_BATT_OUT
Parts:
- BT2: footprint libTX54:BATHLD001TR -> open-lion:BATHLD001TR
- C45, C46, C47: footprint libTX54:VibrationProof_F -> open-lion:VibrationProof_F
- C50, C51, C52, C53, C54, C55: footprint libTX54:SMD_Lytic_E -> open-lion:SMD_Lytic_E
- C56, C57, C58, C59: footprint libTX54:EEEFP0J331AV -> open-lion:EEEFP0J331AV
- D1: value RB068L-40DDTE25 -> B360A-13-F; footprint libTX54:DIOM5226X240N -> open-lion:DIOM5226X240N
- D3, D8, D9: footprint libTX54:SODFL4725X105N -> open-lion:SODFL4725X105N
- D7: footprint libTX54:SODFL1608X70N -> open-lion:SODFL1608X70N
- IC1: footprint libTX54:SOT230P700X180-4N -> open-lion:SOT230P700X180-4N
- IC10: footprint libTX54:SOIC127P600X175-16N -> open-lion:SOIC127P600X175-16N
- IC2: footprint libTX54:SOIC127P1032X265-16N -> open-lion:SOIC127P1032X265-16N
- IC3: footprint libTX54:SOT95P280X145-5N -> open-lion:SOT95P280X145-5N
- IC4: footprint libTX54:SOP65P640X120-16N -> open-lion:SOP65P640X120-16N
- IC5, IC7, IC8: footprint libTX54:SOT65P210X110-5N -> open-lion:SOT65P210X110-5N
- IC6: footprint libTX54:QFP50P900X900X120-49N -> open-lion:QFP50P900X900X120-49N
- IC9: footprint libTX54:SOP50P490X110-10N -> open-lion:SOP50P490X110-10N
- K1: footprint libTX54:G6QE1ADC12 -> open-lion:G6QE1ADC12
- L1, L2: footprint libTX54:B82559A6472A024 -> open-lion:B82559A6472A024
- Q10, Q11, Q12, Q13, Q14, Q5, Q6, Q9: footprint libTX54:LFPAK88 -> open-lion:LFPAK88
- R25, R34, R36, R37, R43: value WSLP40261L000FEA -> GKM5R0010FE-TR; footprint libTX54:WSLP40261L000FEA -> open-lion:WSLP40261L000FEA
- U8: footprint libTX54:AD5663BRMZ-1 -> open-lion:AD5663BRMZ-1
- moved IC8 0.11 mm to (174.7, 108.3)
Connections:
- C2 pad 1: RELAIS_BATT_OUT -> +12P
- C3 pad 1: RELAIS_BATT_OUT -> +12P
- C50 pad 1: RELAIS_BATT_OUT -> +12P
- C51 pad 1: RELAIS_BATT_OUT -> +12P
- C52 pad 1: RELAIS_BATT_OUT -> +12P
- C53 pad 1: RELAIS_BATT_OUT -> +12P
- C54 pad 1: RELAIS_BATT_OUT -> +12P
- C55 pad 1: RELAIS_BATT_OUT -> +12P
- C56 pad 1: RELAIS_BATT_OUT -> +12P
- C57 pad 1: RELAIS_BATT_OUT -> +12P
- C58 pad 1: RELAIS_BATT_OUT -> +12P
- C59 pad 1: RELAIS_BATT_OUT -> +12P
- C60 pad 1: RELAIS_BATT_OUT -> +12P
- C76 pad 1: RELAIS_BATT_OUT -> +12P
- D7 pad 1: ISETA -> GNDA
- D7 pad 2: GNDA -> ISETA
- IC2 pad 1: Net-(IC2-Pad1) -> unconnected-(IC2-32KHZ-Pad1)
- IC2 pad 10: Net-(IC2-Pad10) -> unconnected-(IC2-N.C._6-Pad10)
- IC2 pad 11: Net-(IC2-Pad11) -> unconnected-(IC2-N.C._7-Pad11)
- IC2 pad 12: Net-(IC2-Pad12) -> unconnected-(IC2-N.C._8-Pad12)
- IC2 pad 3: Net-(IC2-Pad3) -> unconnected-(IC2-~{INT}/SQW-Pad3)
- IC2 pad 4: Net-(IC2-Pad4) -> unconnected-(IC2-~{RST}-Pad4)
- IC2 pad 5: Net-(IC2-Pad5) -> unconnected-(IC2-N.C._1-Pad5)
- IC2 pad 6: Net-(IC2-Pad6) -> unconnected-(IC2-N.C._2-Pad6)
- IC2 pad 7: Net-(IC2-Pad7) -> unconnected-(IC2-N.C._3-Pad7)
- IC2 pad 8: Net-(IC2-Pad8) -> unconnected-(IC2-N.C._4-Pad8)
- IC2 pad 9: Net-(IC2-Pad9) -> unconnected-(IC2-N.C._5-Pad9)
- IC3 pad 3: Net-(IC3-Pad3) -> unconnected-(IC3-NC-Pad3)
- IC6 pad 16: Net-(IC6-Pad16) -> unconnected-(IC6-NC_4-Pad16)
- IC6 pad 21: Net-(IC6-Pad21) -> unconnected-(IC6-NC_5-Pad21)
- IC6 pad 3: Net-(IC6-Pad3) -> unconnected-(IC6-NC_1-Pad3)
- IC6 pad 32: Net-(IC6-Pad32) -> unconnected-(IC6-NC_6-Pad32)
- IC6 pad 5: Net-(IC6-Pad5) -> unconnected-(IC6-NC_2-Pad5)
- IC6 pad 6: RELAIS_BATT_OUT -> +12P
- IC6 pad 7: Net-(IC6-Pad7) -> unconnected-(IC6-NC_3-Pad7)
- IC9 pad 3: Net-(IC9-Pad3) -> unconnected-(IC9-NC_1-Pad3)
- IC9 pad 9: Net-(IC9-Pad9) -> unconnected-(IC9-NC_2-Pad9)
- J2 pad 2: RELAIS_BATT_OUT -> +12P
- J9 pad A6: Net-(J9-PadA6) -> unconnected-(J9-D+-PadA6)
- J9 pad A7: Net-(J9-PadA7) -> unconnected-(J9-D--PadA7)
- J9 pad A8: Net-(J9-PadA8) -> unconnected-(J9-SBU1-PadA8)
- J9 pad B6: Net-(J9-PadB6) -> unconnected-(J9-D+-PadB6)
- J9 pad B7: Net-(J9-PadB7) -> unconnected-(J9-D--PadB7)
- J9 pad B8: Net-(J9-PadB8) -> unconnected-(J9-SBU2-PadB8)
- P1 pad 1: Net-(P1-Pad1) -> unconnected-(P1-Pin_1-Pad1)
- P1 pad 4: Net-(P1-Pad4) -> unconnected-(P1-Pin_4-Pad4)
- P2 pad 5: Net-(P2-Pad5) -> unconnected-(P2-Pin_5-Pad5)
- P2 pad 6: Net-(P2-Pad6) -> unconnected-(P2-Pin_6-Pad6)
- P4 pad 7: Net-(P4-Pad7) -> unconnected-(P4-Pin_7-Pad7)
- P4 pad 8: Net-(P4-Pad8) -> unconnected-(P4-Pin_8-Pad8)
- Q10 pad 5: RELAIS_BATT_OUT -> +12P
- Q5 pad 5: RELAIS_BATT_OUT -> +12P
- Q6 pad 5: RELAIS_BATT_OUT -> +12P
- Q9 pad 5: RELAIS_BATT_OUT -> +12P
- U10 pad 2: RELAIS_BATT_OUT -> VBUS
- U9 pad 6: Net-(U9-Pad6) -> unconnected-(U9-NC-Pad6)
- U9 pad 9: Net-(U9-Pad9) -> unconnected-(U9-NC-Pad9)
Routing:
- net RELAIS_BATT_OUT: track 702.2 -> 603.5 mm, vias 52 -> 26
- net +12P: track 0.00 -> 95.8 mm, vias 0 -> 25
- net GNDA: track 172.9 -> 168.8 mm, vias 122 -> 121
- net +5V: track 550.8 -> 548.5 mm
- net GNDPWR: track 134.5 -> 136.2 mm
- net LO1: track 266.0 -> 264.5 mm
- net LO2: track 248.1 -> 246.9 mm
- net HO2: track 254.1 -> 253.0 mm
- net CS1B: track 118.2 -> 117.3 mm
- net ISETA: track 72.2 -> 72.9 mm, vias 6 -> 7
- net 11_MOSI: vias 5 -> 4
- added copper zone on In1.Cu, net +12P
- added copper zone on In1.Cu, net BATT+_CHARGE
- added copper zone on In1.Cu, net GNDA
- added copper zone on In2.Cu, net GNDA
- added copper zone on In1.Cu, net GNDPWR
- added copper zone on In2.Cu, net GNDPWR
- added copper zone on In1.Cu, net Net-(BT1-+)
- added copper zone on In1.Cu, net Net-(BT1--)
- added copper zone on In1.Cu, net Net-(L1-Pad2)
- added copper zone on In1.Cu, net SW1
- added copper zone on In1.Cu, net SW2
- added copper zone on In1.Cu, net TO_SHUNT_CHARGE
Other:
- copper layers 2 -> 4
- board text added: "OPEN-LION-CHARGER APE 2025"
- board text removed: "BANC D'ESSAI LITHIUM ION TX54 - A21 REV 2.0"
