File: hw/open-lion-charger/open-lion-charger.kicad_pcb (KiCad board)
At the start: 4 copper layers, 139.7 x 186 mm, 235 parts, among them IC1 MCP1799-3302H_DB, IC10 MUX509IDR, IC2 DS3231M+TRL, IC3 TMP36GRTZ-REEL7, IC4 ADS122C04IPWR, IC5 INA280A3IDCKR, IC6 LM5170QPHPTQ1, IC7 INA280A3IDCKR, IC8 INA280A3IDCKR, IC9 DAC80501MDGSR, J1 Barrel_Jack_Switch, J2 Conn_01x02_Female, J3 Conn_01x02_Female, J4 Conn_01x06_Female, J5 Conn_01x02_Female, J6 Conn_01x02_Female, J8 Conn_01x02_Female, J9 USB_C_Receptacle, K1 G6QE-1A_DC12, P1 Power, P2 Analog, P3 Digital, P4 Digital, Q1 PBHV9115TLH, Q10 PSMNR55-40SSHJ, Q11 PSMNR55-40SSHJ, Q12 PSMNR55-40SSHJ, Q13 PSMNR55-40SSHJ, Q14 PSMNR55-40SSHJ, Q2 SiS176LDN, Q3 PBHV8115T, Q4 PBHV8115T, Q5 PSMNR55-40SSHJ, Q6 PSMNR55-40SSHJ, Q7 IXTH30N50L2, Q8 IXTH30N50L2, Q9 PSMNR55-40SSHJ, U1 LM1117-5.0, U10 FUSB302T, U2 MAX31855JASA, U3 MAX31855JASA, U4 TLV9151SIDBVR, U5 TLV9151SIDBVR, U6 LMP7701, U7 LMP7701, U8 AD5663BRMZ-1, U9 MAX3377EEUD+

Commit message: Prepare for fab
Parts:
- added NT1: NetTie_2, Resistor_SMD:R_2816_7142Metric_Pad3.20x4.45mm_HandSolder, B.Cu at (195.1, 45.1)
- moved NT2 0.38 mm to (89.5, 92.8)
- turned D7 to -90 degrees
Connections:
- C77 pad 1: RELAIS_BATT_OUT -> VBUS
- J9 pad A4: RELAIS_BATT_OUT -> VBUS
- J9 pad A9: RELAIS_BATT_OUT -> VBUS
- J9 pad B4: RELAIS_BATT_OUT -> VBUS
- J9 pad B9: RELAIS_BATT_OUT -> VBUS
- TP11 pad 1: RELAIS_BATT_OUT -> VBUS
- TP2 pad 1: RELAIS_BATT_OUT -> +12P
Routing:
- net RELAIS_BATT_OUT: track 603.5 -> 503.5 mm
- net VBUS: track 0.00 -> 39.0 mm
- net +12P: track 95.8 -> 104.9 mm
- net GNDA: track 168.8 -> 175.3 mm, vias 121 -> 123
- net SW2: track 195.8 -> 194.1 mm
- net LO2: track 246.9 -> 245.3 mm
- net HO2: track 253.0 -> 251.6 mm
- net HO1: track 257.1 -> 255.9 mm
- net LO1: track 264.5 -> 263.5 mm
- net Net-(Q7-G): track 236.7 -> 235.9 mm
- net ISETA: track 72.9 -> 72.2 mm, vias 7 -> 6
- net Net-(IC8-IN+): track 194.3 -> 193.8 mm
- added copper zone on B.Cu, net +12P
- added copper zone on F.Cu, net VBUS
- removed copper zone on B.Cu, net RELAIS_BATT_OUT
