File: hw/open-lion-charger/Arduino.kicad_sch (KiCad schematic)
At the start: 25 parts, among them J3 Conn_01x02_Female, J4 Conn_01x06_Female, P1 Power, P2 Analog, P3 Digital, P4 Digital, Q3 PBHV8115T, Q4 PBHV8115T, U10 FUSB302T

Commit message: Done with PCB review
Warning : issue with net +12P and confusion with RELAIS_BATT_OUT
Parts:
- D3: footprint SODFL4725X105N -> open-lion:SODFL4725X105N
Changed lines of the file:
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@@
 			)
 		)
-		(property "Footprint" "SODFL4725X105N"
+		(property "Footprint" "open-lion:SODFL4725X105N"
 			(at 69.088 43.942 0)
 			(effects
