File: hw/open-lion-charger/Power.kicad_sch (KiCad schematic)
At the start: 30 parts, among them IC1 MCP1799-3302H_DB, J1 Barrel_Jack_Switch, J2 Conn_01x02_Female, J7 Conn_01x02_Female, J8 Conn_01x02_Female, J9 USB_C_Receptacle, K1 G6QE-1A_DC12, Q1 PBHV9115TLH, Q2 SiS176LDN, U1 LM1117-5.0

Commit message: Done with PCB review
Warning : issue with net +12P and confusion with RELAIS_BATT_OUT
Parts:
- D1: footprint DIOM5226X240N -> open-lion:DIOM5226X240N
- IC1: footprint SOT230P700X180-4N -> open-lion:SOT230P700X180-4N
- J7: now not fitted
- K1: footprint SamacSys_OLD:G6QE1ADC12 -> open-lion:G6QE1ADC12
Changed lines of the file:
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@@
 	)
 	(junction
-		(at 53.975 73.025)
+		(at 55.88 46.99)
 		(diameter 0)
 		(color 0 0 0 0)
 	)
 	(junction
-		(at 238.76 30.734)
+		(at 53.975 73.025)
 		(diameter 0)
 		(color 0 0 0 0)
 	)
 	(junction
-		(at 96.52 155.702)
+		(at 238.76 30.734)
 		(diameter 0)
 		(color 0 0 0 0)
 	)
 	(junction
-		(at 86.614 46.99)
+		(at 96.52 155.702)
 		(diameter 0)
 		(color 0 0 0 0)
@@
 	)
 	(junction
-		(at 130.556 115.57)
+		(at 86.614 46.99)
 		(diameter 0)
 		(color 0 0 0 0)
 	)
 	(junction
-		(at 173.228 30.48)
+		(at 130.556 115.57)
 		(diameter 0)
 		(color 0 0 0 0)
 	)
 	(junction
-		(at 243.078 92.329)
+		(at 173.228 30.48)
 		(diameter 0)
 		(color 0 0 0 0)
 	)
 	(junction
-		(at 111.252 115.57)
+		(at 243.078 92.329)
 		(diameter 0)
 		(color 0 0 0 0)
 	)
 	(junction
-		(at 55.88 46.99)
+		(at 111.252 115.57)
 		(diameter 0)
 		(color 0 0 0 0)
@@
 	(wire
 		(pts
+			(xy 55.88 46.99) (xy 86.614 46.99)
+		)
+		(stroke
+			(width 0)
+			(type default)
+		)
+	)
+	(wire
+		(pts
 			(xy 93.853 176.276) (xy 153.162 176.276)
 		)
@@
 	(wire
 		(pts
-			(xy 86.614 46.99) (xy 99.06 46.99)
-		)
-		(stroke
-			(width 0)
-			(type default)
-		)
-	)
-	(wire
-		(pts
 			(xy 50.165 75.565) (xy 50.165 78.105)
 		)
@@
 	(wire
 		(pts
+			(xy 86.614 46.99) (xy 99.06 46.99)
+		)
+		(stroke
+			(width 0)
+			(type default)
+		)
+	)
+	(wire
+		(pts
 			(xy 173.228 30.48) (xy 173.228 33.02)
 		)
@@
 		)
 	)
-	(wire
-		(pts
-			(xy 55.88 46.99) (xy 86.614 46.99)
-		)
-		(stroke
-			(width 0)
-			(type default)
-		)
-	)
 	(text "Alimentation à découpage\n12V, 12.5A max"
 		(exclude_from_sim no)
@@
 			)
 		)
-		(property "Footprint" "DIOM5226X240N"
+		(property "Footprint" "open-lion:DIOM5226X240N"
 			(at 130.556 127.254 0)
 			(effects
@@
 			)
 		)
-		(property "Footprint" "SOT230P700X180-4N"
+		(property "Footprint" "open-lion:SOT230P700X180-4N"
 			(at 268.986 29.21 0)
 			(effects
@@
 			)
 		)
-		(property "Footprint" "SamacSys_OLD:G6QE1ADC12"
+		(property "Footprint" "open-lion:G6QE1ADC12"
 			(at 69.85 107.95 0)
 			(effects
@@
 		(exclude_from_sim no)
 		(in_bom yes)
-		(on_board yes)
-		(dnp no)
+		(on_board no)
+		(dnp yes)
 		(property "Reference" "J7"
 			(at 39.37 44.45 0)

Commit message: Prepare for fab
Parts:
- added NT1: NetTie_2, Resistor_SMD:R_2816_7142Metric_Pad3.20x4.45mm_HandSolder, symbol Device:NetTie_2
Connections:
- net +12P: no longer C1.1, C4.1, C6.1, C77.1, IC1.1 (VIN), J1.1, J9.A4 (VBUS), J9.A9 (VBUS), J9.B4 (VBUS), J9.B9 (VBUS), TP1.1, TP11.1, U1.3 (VI)
- new net +12V: C1.1, C4.1, C6.1, IC1.1 (VIN), J1.1, NT1.2, TP1.1, U1.3 (VI)
- new net VBUS: C77.1, J9.A4 (VBUS), J9.A9 (VBUS), J9.B4 (VBUS), J9.B9 (VBUS), NT1.1, TP11.1
Other:
- moved on the sheet: TP11
